File: atmega88_based_pcb/atmega88_based_pcb.kicad_sch (KiCad schematic)
At the start: 65 parts, among them J1 Barrel_Jack, J2 USB_A, J3 Screw_Terminal_01x04, SW1 SW_Push, U1 ATmega168-20P, U10 SC56-11SURKWA, U11 SC56-11SURKWA, U12 SC56-11SURKWA, U13 SC56-11SURKWA, U2 LM1084-5.0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

Commit message: Tied AVCC to VCC and changed interrupt pins to use PD3/4 for external interrupts instead of PCINT
Parts:
- TP1, TP2, TP3, TP4, TP5: footprint TestPoint:TestPoint_Pad_1.0x1.0mm -> footprint_library:TestPoint_Pad_1.0x1.0mm_wide
Connections:
- net VCC: now also U1.20 (AVCC)
- net at C3.2, D1.1 (K), J3.3 (Pin_3)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: now also U1.6 (PD4); no longer U1.3 (PD1)
- net at C4.2, D2.1 (K), J3.1 (Pin_1)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: now also U1.5 (PD3); no longer U1.2 (PD0)
- no-connect marks 21 -> 18
Changed lines of the file:
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@@
 	)
 	(junction
+		(at 45.72 68.58)
+		(diameter 0)
+		(color 0 0 0 0)
+	)
+	(junction
 		(at 76.2 175.26)
 		(diameter 0)
@@
 	)
 	(no_connect
-		(at 48.26 69.85)
-	)
-	(no_connect
 		(at 167.64 116.84)
 	)
@@
 	)
 	(no_connect
-		(at 60.96 130.81)
-	)
-	(no_connect
 		(at 60.96 133.35)
 	)
@@
 	)
 	(no_connect
-		(at 60.96 128.27)
-	)
-	(no_connect
 		(at 60.96 95.25)
 	)
@@
 	(wire
 		(pts
+			(xy 60.96 128.27) (xy 76.2 128.27)
+		)
+		(stroke
+			(width 0)
+			(type default)
+		)
+	)
+	(wire
+		(pts
 			(xy 132.08 33.02) (xy 134.62 33.02)
 		)
@@
 	(wire
 		(pts
-			(xy 45.72 66.04) (xy 45.72 69.85)
+			(xy 45.72 66.04) (xy 45.72 68.58)
 		)
 		(stroke
@@
 	(wire
 		(pts
-			(xy 71.12 123.19) (xy 60.96 123.19)
-		)
-		(stroke
-			(width 0)
-			(type default)
-		)
-	)
-	(wire
-		(pts
 			(xy 54.61 55.88) (xy 45.72 55.88)
 		)
@@
 	(wire
 		(pts
-			(xy 58.42 157.48) (xy 64.77 157.48)
+			(xy 60.96 130.81) (xy 71.12 130.81)
 		)
 		(stroke
@@
 	(wire
 		(pts
-			(xy 138.43 77.47) (xy 140.97 77.47)
+			(xy 58.42 157.48) (xy 64.77 157.48)
 		)
 		(stroke
@@
 	(wire
 		(pts
-			(xy 154.94 106.68) (xy 157.48 106.68)
+			(xy 138.43 77.47) (xy 140.97 77.47)
 		)
 		(stroke
@@
 	(wire
 		(pts
-			(xy 45.72 35.56) (xy 48.26 35.56)
+			(xy 154.94 106.68) (xy 157.48 106.68)
 		)
 		(stroke
@@
 	(wire
 		(pts
-			(xy 148.59 80.01) (xy 151.13 80.01)
+			(xy 45.72 35.56) (xy 48.26 35.56)
 		)
 		(stroke
@@
 	(wire
 		(pts
-			(xy 138.43 80.01) (xy 140.97 80.01)
+			(xy 148.59 80.01) (xy 151.13 80.01)
 		)
 		(stroke
@@
 	(wire
 		(pts
-			(xy 83.82 100.33) (xy 83.82 106.68)
+			(xy 138.43 80.01) (xy 140.97 80.01)
 		)
 		(stroke
@@
 	(wire
 		(pts
-			(xy 54.61 52.07) (xy 54.61 55.88)
+			(xy 83.82 100.33) (xy 83.82 106.68)
 		)
 		(stroke
@@
 	(wire
 		(pts
-			(xy 76.2 120.65) (xy 76.2 146.05)
+			(xy 54.61 52.07) (xy 54.61 55.88)
 		)
 		(stroke
@@
 	(wire
 		(pts
-			(xy 76.2 120.65) (xy 60.96 120.65)
-		)
-		(stroke
-			(width 0)
-			(type default)
-		)
-	)
-	(wire
-		(pts
 			(xy 63.5 115.57) (xy 60.96 115.57)
 		)
@@
 	(wire
 		(pts
-			(xy 71.12 123.19) (xy 71.12 146.05)
+			(xy 172.72 142.24) (xy 175.26 142.24)
 		)
 		(stroke
@@
 	(wire
 		(pts
-			(xy 172.72 142.24) (xy 175.26 142.24)
+			(xy 48.26 69.85) (xy 48.26 68.58)
 		)
 		(stroke
@@
 	(wire
 		(pts
+			(xy 45.72 68.58) (xy 48.26 68.58)
+		)
+		(stroke
+			(width 0)
+			(type default)
+		)
+	)
+	(wire
+		(pts
 			(xy 182.88 137.16) (xy 185.42 137.16)
 		)
@@
 	(wire
 		(pts
+			(xy 45.72 68.58) (xy 45.72 69.85)
+		)
+		(stroke
+			(width 0)
+			(type default)
+		)
+	)
+	(wire
+		(pts
 			(xy 138.43 82.55) (xy 140.97 82.55)
 		)
@@
 		)
 	)
+	(wire
+		(pts
+			(xy 71.12 130.81) (xy 71.12 146.05)
+		)
+		(stroke
+			(width 0)
+			(type default)
+		)
+	)
+	(wire
+		(pts
+			(xy 76.2 128.27) (xy 76.2 146.05)
+		)
+		(stroke
+			(width 0)
+			(type default)
+		)
+	)
 	(label "BCD_INPUT_D"
 		(at 96.52 48.26 180)
@@
 			)
 		)
-		(property "Footprint" "TestPoint:TestPoint_Pad_1.0x1.0mm"
+		(property "Footprint" "footprint_library:TestPoint_Pad_1.0x1.0mm_wide"
 			(at 71.12 140.97 0)
 			(effects
@@
 			)
 		)
-		(property "Footprint" "TestPoint:TestPoint_Pad_1.0x1.0mm"
+		(property "Footprint" "footprint_library:TestPoint_Pad_1.0x1.0mm_wide"
 			(at 76.2 151.13 0)
 			(effects
@@
 			)
 		)
-		(property "Footprint" "TestPoint:TestPoint_Pad_1.0x1.0mm"
+		(property "Footprint" "footprint_library:TestPoint_Pad_1.0x1.0mm_wide"
 			(at 58.42 115.57 0)
 			(effects
@@
 			)
 		)
-		(property "Footprint" "TestPoint:TestPoint_Pad_1.0x1.0mm"
+		(property "Footprint" "footprint_library:TestPoint_Pad_1.0x1.0mm_wide"
 			(at 59.69 60.96 0)
 			(effects
@@
 			)
 		)
-		(property "Footprint" "TestPoint:TestPoint_Pad_1.0x1.0mm"
+		(property "Footprint" "footprint_library:TestPoint_Pad_1.0x1.0mm_wide"
 			(at 68.58 26.67 0)
 			(effects

Commit message: Added some page metadata to schematic
Other:
- title: (none) -> Speed'o'Matic
Changed lines of the file:
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@@
 	(generator_version "9.0")
 	(paper "A4")
+	(title_block
+		(title "Speed'o'Matic")
+		(date "2025-04-24")
+		(rev "2")
+		(comment 1 "TODO: Replace USB-A receptacle")
+		(comment 2 "Optional debounce caps for barriers included")
+		(comment 4 "Uses a seperate driver IC for every digit")
+	)
 	(text "Optional\ndebounce capacitcance"
 		(exclude_from_sim no)
